File: omni_pcb.kicad_pcb (KiCad board)
At the start: 2 copper layers, 25 parts, among them J1 Conn_01x06_Socket, J2 Conn_01x06_Socket, J3 Conn_01x06_Socket, J4 Conn_01x06_Socket, U1 ESP32-DEVKIT-V1

Commit message: pcb layout
Parts:
- removed J1, J2, J3, J4: Conn_01x06_Socket, Connector_JST:JST_XH_B6B-XH-AM_1x06_P2.50mm_Vertical
- removed MD_L1, MD_L2, MD_L3, MD_L4, MD_R1, MD_R2, MD_R3, MD_R4: Conn_01x04_Socket, Connector_PinSocket_1.00mm:PinSocket_1x04_P1.00mm_Vertical
- removed U1: ESP32-DEVKIT-V1, ESP32-WROOM-V1_30pins:MODULE_ESP32_DEVKIT_V1
- removed pow-M1, pow-M2, pow-M3, pow-M4, pow-M5, pow-M6, pow-M7, pow-M8: Screw_Terminal_01x02, TerminalBlock:TerminalBlock_Xinya_XY308-2.54-2P_1x02_P2.54mm_Horizontal
- added Alt_enc1: Conn_01x06_Socket, Connector_JST:JST_XH_B6B-XH-AM_1x06_P2.50mm_Vertical, F.Cu at (178.0, 40.0)
- added Alt_enc2: Conn_01x06_Socket, Connector_JST:JST_XH_B6B-XH-AM_1x06_P2.50mm_Vertical, F.Cu at (122.3, 35.5)
- added Alt_enc3: Conn_01x06_Socket, Connector_JST:JST_XH_B6B-XH-AM_1x06_P2.50mm_Vertical, F.Cu at (190.5, 85.5)
- added Alt_enc4: Conn_01x06_Socket, Connector_JST:JST_XH_B6B-XH-AM_1x06_P2.50mm_Vertical, F.Cu at (134.8, 88.0)
- added ESP1: ESP, ESP32-WROOM-V1_30pins:MODULE_ESP32_DEVKIT_V1, F.Cu at (169.2, 62.7)
- added ESP_5V1: ESP_5V, Connector_PinHeader_2.54mm:PinHeader_1x01_P2.54mm_Vertical, F.Cu at (153.8, 62.5)
- added Enc1: Conn_01x06_Socket, Connector_JST:JST_XH_B6B-XH-AM_1x06_P2.50mm_Vertical, F.Cu at (158.8, 40.0)
- added Enc2: Conn_01x06_Socket, Connector_JST:JST_XH_B6B-XH-AM_1x06_P2.50mm_Vertical, F.Cu at (122.3, 43.7)
- added Enc3: Conn_01x06_Socket, Connector_JST:JST_XH_B6B-XH-AM_1x06_P2.50mm_Vertical, F.Cu at (171.3, 85.5)
- added Enc4: Conn_01x06_Socket, Connector_JST:JST_XH_B6B-XH-AM_1x06_P2.50mm_Vertical, F.Cu at (134.8, 80.0)
- added Ext_12V1: Ext_12V, Connector_PinHeader_2.54mm:PinHeader_1x01_P2.54mm_Vertical, F.Cu at (82.9, 94.5)
- added Ext_5V1: Ext_5V, Connector_PinHeader_2.54mm:PinHeader_1x01_P2.54mm_Vertical, F.Cu at (147.1, 62.6)
- added Ext_GND1: Ext_GND, Connector_PinHeader_2.54mm:PinHeader_1x01_P2.54mm_Vertical, F.Cu at (82.9, 29.1)
- added G***: LOGO, Logo:atom_logo, F.Cu at (137.0, 60.6)
- added H1: MountingHole, MountingHole:MountingHole_2.5mm, F.Cu at (191.5, 99.8)
- added H2: MountingHole, MountingHole:MountingHole_2.5mm, F.Cu at (83.1, 99.8)
- added H3: MountingHole, MountingHole:MountingHole_2.5mm, F.Cu at (191.5, 23.7)
- added H4: MountingHole, MountingHole:MountingHole_2.5mm, F.Cu at (83.0, 23.6)
- added MD1: Conn_02x04_Odd_Even, Connector_PinSocket_2.54mm:PinSocket_2x04_P2.54mm_Vertical, F.Cu at (122.6, 22.2)
- added MD2: Conn_02x04_Odd_Even, Connector_PinSocket_2.54mm:PinSocket_2x04_P2.54mm_Vertical, F.Cu at (178.1, 22.2)
- added MD3: Conn_02x04_Odd_Even, Connector_PinSocket_2.54mm:PinSocket_2x04_P2.54mm_Vertical, F.Cu at (153.8, 101.2)
- added MD4: Conn_02x04_Odd_Even, Connector_PinSocket_2.54mm:PinSocket_2x04_P2.54mm_Vertical, F.Cu at (100.2, 101.2)
- added MD_st1: Conn_01x04, Connector_JST:JST_XH_B4B-XH-A_1x04_P2.50mm_Vertical, F.Cu at (144.0, 40.0)
- added MD_st2: Conn_01x04, Connector_JST:JST_XH_B4B-XH-A_1x04_P2.50mm_Vertical, F.Cu at (112.8, 43.1)
- added MD_st3: Conn_01x04, Connector_JST:JST_XH_B4B-XH-A_1x04_P2.50mm_Vertical, F.Cu at (151.5, 85.5)
- added MD_st4: Conn_01x04, Connector_JST:JST_XH_B4B-XH-A_1x04_P2.50mm_Vertical, F.Cu at (113.0, 87.9)
- B-SW_1: value 100SP1T1B4M2QE -> SW
- Bin1: value Battery_Terminal -> Bin
- IMU1: value Conn_01x08_Socket -> IMU; footprint Connector_PinSocket_1.00mm:PinSocket_1x08_P1.00mm_Vertical -> Connector_PinSocket_2.54mm:PinSocket_1x10_P2.54mm_Vertical
- moved Bin1 42.8 mm to (83.3, 86.6), turned to -90 degrees
- moved BUCK1 40.5 mm to (107.0, 82.6)
- moved B-SW_1 29.9 mm to (97.7, 88.1), turned to -90 degrees
- moved IMU1 29.6 mm to (113.2, 73.2), turned to 180 degrees
Connections:
- IMU1 pad 5: /SDA_imu -> unconnected-(IMU1-Pin_5-Pad5)
- IMU1 pad 6: /SCL_imu -> unconnected-(IMU1-Pin_6-Pad6)
- IMU1 pad 7: GND -> /SDA_imu
- IMU1 pad 8: +5V -> /SCL_imu
Other:
- board outline added: 116.5 x 84.2 mm
- board text added: "A.T.O.M. Robotics"

Commit message: traces
Parts:
- removed G***: LOGO, Logo:atom_logo
- added atom: LOGO, Logo:atom_logo_20x20mm, F.Cu at (134.7, 58.0)
- ESP_5V1, Ext_5V1: footprint Connector_PinHeader_2.54mm:PinHeader_1x01_P2.54mm_Vertical -> Connector_Wire:SolderWirePad_1x01_SMD_2x4mm
- Ext_12V1, Ext_GND1: footprint Connector_PinHeader_2.54mm:PinHeader_1x01_P2.54mm_Vertical -> Connector_Wire:SolderWirePad_1x01_SMD_3x6mm
- moved Alt_enc1 12.7 mm to (190.6, 41.1), turned to 180 degrees
- moved Enc1 12.6 mm to (171.4, 41.1), turned to 180 degrees
- moved MD_st1 7.58 mm to (151.5, 41.1), turned to 180 degrees
- moved Ext_5V1 7.35 mm to (153.8, 65.6), turned to -90 degrees
- moved H1 0.68 mm to (191.5, 100.5)
- moved H2 0.67 mm to (83.1, 100.4)
- moved ESP_5V1 0.65 mm to (153.8, 61.9), turned to -90 degrees
- moved H4 0.60 mm to (83.0, 23.0)
- moved Ext_12V1 0.34 mm to (83.0, 94.2), turned to -90 degrees
- moved Ext_GND1 0.12 mm to (83.0, 29.2), turned to -90 degrees
Connections:
- Alt_enc1 pad 1: unconnected-(Alt_enc1-Pin_1-Pad1) -> /M+1
- Alt_enc1 pad 2: unconnected-(Alt_enc1-Pin_2-Pad2) -> +5V
- Alt_enc1 pad 3: unconnected-(Alt_enc1-Pin_3-Pad3) -> /M1_ChB
- Alt_enc1 pad 4: unconnected-(Alt_enc1-Pin_4-Pad4) -> /M1_ChA
- Alt_enc1 pad 5: unconnected-(Alt_enc1-Pin_5-Pad5) -> GND
- Alt_enc1 pad 6: unconnected-(Alt_enc1-Pin_6-Pad6) -> /M-1
- Alt_enc2 pad 1: unconnected-(Alt_enc2-Pin_1-Pad1) -> /M+2
- Alt_enc2 pad 2: unconnected-(Alt_enc2-Pin_2-Pad2) -> +5V
- Alt_enc2 pad 3: unconnected-(Alt_enc2-Pin_3-Pad3) -> /M2_ChB
- Alt_enc2 pad 4: unconnected-(Alt_enc2-Pin_4-Pad4) -> /M2_ChA
- Alt_enc2 pad 5: unconnected-(Alt_enc2-Pin_5-Pad5) -> GND
- Alt_enc2 pad 6: unconnected-(Alt_enc2-Pin_6-Pad6) -> /M-2
- Alt_enc3 pad 1: unconnected-(Alt_enc3-Pin_1-Pad1) -> /M+3
- Alt_enc3 pad 2: unconnected-(Alt_enc3-Pin_2-Pad2) -> +5V
- Alt_enc3 pad 3: unconnected-(Alt_enc3-Pin_3-Pad3) -> /M3_ChB
- Alt_enc3 pad 4: unconnected-(Alt_enc3-Pin_4-Pad4) -> /M3_ChA
- Alt_enc3 pad 5: unconnected-(Alt_enc3-Pin_5-Pad5) -> GND
- Alt_enc3 pad 6: unconnected-(Alt_enc3-Pin_6-Pad6) -> /M-3
- Alt_enc4 pad 1: unconnected-(Alt_enc4-Pin_1-Pad1) -> /M+4
- Alt_enc4 pad 2: unconnected-(Alt_enc4-Pin_2-Pad2) -> +5V
- Alt_enc4 pad 3: unconnected-(Alt_enc4-Pin_3-Pad3) -> /M4_ChB
- Alt_enc4 pad 4: unconnected-(Alt_enc4-Pin_4-Pad4) -> /M4_ChA
- Alt_enc4 pad 5: unconnected-(Alt_enc4-Pin_5-Pad5) -> GND
- Alt_enc4 pad 6: unconnected-(Alt_enc4-Pin_6-Pad6) -> /M-4
- ESP1 pad 10: /L_PWM_3 -> /M3_ChB
- ESP1 pad 21: /R_PWM_1 -> /R_PWM_2
- ESP1 pad 22: /L_PWM_1 -> /L_PWM_2
- ESP1 pad 23: /M2_ChB -> /R_PWM_1
- ESP1 pad 24: /M2_ChA -> /L_PWM_1
- ESP1 pad 25: /R_PWM_2 -> /M2_ChA
- ESP1 pad 26: /L_PWM_2 -> /M2_ChB
- ESP1 pad 27: /M4_ChA -> /M4_ChB
- ESP1 pad 28: /M4_ChB -> /M4_ChA
- ESP1 pad 5: /M3_ChB -> /R_PWM_3
- ESP1 pad 8: /M3_ChA -> /L_PWM_3
- ESP1 pad 9: /R_PWM_3 -> /M3_ChA
Routing:
- net +5V: track 0.00 -> 568.2 mm
- net /Vin: track 0.00 -> 182.4 mm
- net /R_PWM_4: track 0.00 -> 86.9 mm
- net /SCL_imu: track 0.00 -> 82.8 mm
- net /L_PWM_4: track 0.00 -> 81.3 mm
- net /SDA_imu: track 0.00 -> 74.3 mm
- net /M4_ChA: track 0.00 -> 61.0 mm
- net /R_PWM_1: track 0.00 -> 60.7 mm
- net /M4_ChB: track 0.00 -> 60.3 mm
- net /L_PWM_1: track 0.00 -> 57.0 mm
- net /M2_ChB: track 0.00 -> 55.7 mm
- net /M2_ChA: track 0.00 -> 55.3 mm
- net /M+3: track 0.00 -> 48.4 mm
- net /M+1: track 0.00 -> 46.4 mm
- net /M-2: track 0.00 -> 44.7 mm
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- added copper zone on F.Cu, net GND
Other:
- board size 116.5 x 84.2 mm -> 116.5 x 85.5 mm

Commit message: traces
Routing:
- net GND: vias 0 -> 40
- added copper zone on B.Cu, net GND

Commit message: pcb final
Parts:
- Alt_enc1, Alt_enc2, Alt_enc3, Alt_enc4, Enc1, Enc2, Enc3, Enc4: footprint Connector_JST:JST_XH_B6B-XH-AM_1x06_P2.50mm_Vertical -> Connector_JST:JST_XH_B6B-XH-A_1x06_P2.50mm_Vertical
- moved Alt_enc1 12.7 mm to (177.9, 40.1), turned to 0 degrees
- moved Enc1 12.7 mm to (158.8, 40.1), turned to 0 degrees
- moved MD_st1 7.57 mm to (144.0, 40.1), turned to 0 degrees
- moved ESP_5V1 4.15 mm to (153.7, 57.7)
- moved Ext_5V1 3.75 mm to (153.7, 61.9)
- moved H4 1.30 mm to (83.0, 24.3)
- moved Bin1 1.29 mm to (83.5, 85.3)
- moved H1 1.25 mm to (191.6, 99.2)
- moved H2 1.25 mm to (83.1, 99.2)
- moved B-SW_1 1.18 mm to (97.7, 86.9)
- moved Ext_12V1 0.87 mm to (83.4, 93.4)
- moved H3 0.60 mm to (191.6, 24.3)
- moved Ext_GND1 0.40 mm to (83.4, 29.2)
Connections:
- Alt_enc1 pad 1: /M+1 -> unconnected-(Alt_enc1-Pin_1-Pad1)
- Alt_enc1 pad 2: +5V -> unconnected-(Alt_enc1-Pin_2-Pad2)
- Alt_enc1 pad 3: /M1_ChB -> unconnected-(Alt_enc1-Pin_3-Pad3)
- Alt_enc1 pad 4: /M1_ChA -> unconnected-(Alt_enc1-Pin_4-Pad4)
- Alt_enc1 pad 5: GND -> unconnected-(Alt_enc1-Pin_5-Pad5)
- Alt_enc1 pad 6: /M-1 -> unconnected-(Alt_enc1-Pin_6-Pad6)
- Alt_enc2 pad 1: /M+2 -> unconnected-(Alt_enc2-Pin_1-Pad1)
- Alt_enc2 pad 2: +5V -> unconnected-(Alt_enc2-Pin_2-Pad2)
- Alt_enc2 pad 3: /M2_ChB -> unconnected-(Alt_enc2-Pin_3-Pad3)
- Alt_enc2 pad 4: /M2_ChA -> unconnected-(Alt_enc2-Pin_4-Pad4)
- Alt_enc2 pad 5: GND -> unconnected-(Alt_enc2-Pin_5-Pad5)
- Alt_enc2 pad 6: /M-2 -> unconnected-(Alt_enc2-Pin_6-Pad6)
- Alt_enc3 pad 1: /M+3 -> unconnected-(Alt_enc3-Pin_1-Pad1)
- Alt_enc3 pad 2: +5V -> unconnected-(Alt_enc3-Pin_2-Pad2)
- Alt_enc3 pad 3: /M3_ChB -> unconnected-(Alt_enc3-Pin_3-Pad3)
- Alt_enc3 pad 4: /M3_ChA -> unconnected-(Alt_enc3-Pin_4-Pad4)
- Alt_enc3 pad 5: GND -> unconnected-(Alt_enc3-Pin_5-Pad5)
- Alt_enc3 pad 6: /M-3 -> unconnected-(Alt_enc3-Pin_6-Pad6)
- Alt_enc4 pad 1: /M+4 -> unconnected-(Alt_enc4-Pin_1-Pad1)
- Alt_enc4 pad 2: +5V -> unconnected-(Alt_enc4-Pin_2-Pad2)
- Alt_enc4 pad 3: /M4_ChB -> unconnected-(Alt_enc4-Pin_3-Pad3)
- Alt_enc4 pad 4: /M4_ChA -> unconnected-(Alt_enc4-Pin_4-Pad4)
- Alt_enc4 pad 5: GND -> unconnected-(Alt_enc4-Pin_5-Pad5)
- Alt_enc4 pad 6: /M-4 -> unconnected-(Alt_enc4-Pin_6-Pad6)
- ESP1 pad 19: /M1_ChB -> /R_PWM_2
- ESP1 pad 20: /M1_ChA -> /L_PWM_2
- ESP1 pad 21: /R_PWM_2 -> /M1_ChA
- ESP1 pad 22: /L_PWM_2 -> /M1_ChB
- MD1 pad 2: +5V -> GND
- MD2 pad 2: +5V -> GND
- MD3 pad 2: +5V -> GND
- MD4 pad 2: +5V -> GND
Routing:
- net +5V: track 568.2 -> 475.2 mm
- net /M+3: track 48.4 -> 14.1 mm
- net /M+4: track 39.6 -> 15.8 mm
- net /M-3: track 36.2 -> 13.2 mm
- net /M3_ChA: track 31.1 -> 12.3 mm
- net /M3_ChB: track 30.5 -> 12.3 mm
- net /M+2: track 39.3 -> 25.2 mm
- net /M+1: track 46.4 -> 32.4 mm
- net /M-4: track 22.8 -> 11.5 mm
- net /M2_ChB: track 55.7 -> 45.5 mm
- net /M2_ChA: track 55.3 -> 45.1 mm
- net /M4_ChB: track 60.3 -> 50.2 mm
- net /M4_ChA: track 61.0 -> 50.9 mm
- net /Vin: track 182.4 -> 191.1 mm
- net /M-2: track 44.7 -> 36.3 mm
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Other:
- board size 116.5 x 85.5 mm -> 116.6 x 82.9 mm

Commit message: pin changes
Parts:
- moved Alt_enc1 19.4 mm to (158.6, 40.0)
- moved Enc3 19.2 mm to (190.5, 85.5)
- moved Enc1 19.2 mm to (177.9, 40.1)
- moved Alt_enc3 19.0 mm to (171.4, 85.5)
Connections:
- ESP1 pad 10: /M3_ChB -> /M3_ChA
- ESP1 pad 15: unconnected-(ESP1-D23-Pad15) -> /M3_ChB
- ESP1 pad 19: /R_PWM_2 -> /M1_ChA
- ESP1 pad 20: /L_PWM_2 -> /M1_ChB
- ESP1 pad 21: /M1_ChA -> /R_PWM_2
- ESP1 pad 22: /M1_ChB -> /L_PWM_2
- ESP1 pad 27: /M4_ChB -> /M4_ChA
- ESP1 pad 28: /M4_ChA -> /R_PWM_4
- ESP1 pad 3: /R_PWM_4 -> /L_PWM_4
- ESP1 pad 4: /L_PWM_4 -> /R_PWM_3
- ESP1 pad 5: /R_PWM_3 -> /L_PWM_3
- ESP1 pad 8: /L_PWM_3 -> unconnected-(ESP1-D5-Pad8)
- ESP1 pad 9: /M3_ChA -> /M4_ChB
Routing:
- net /M+1: track 32.4 -> 52.0 mm
- net /M-1: track 31.3 -> 50.9 mm
- net /M-3: track 13.2 -> 32.7 mm
- net /M+3: track 14.1 -> 33.6 mm
- net /R_PWM_4: track 89.8 -> 109.2 mm
- net +5V: track 475.2 -> 492.8 mm
- net /M1_ChB: track 22.0 -> 10.4 mm
- net /M1_ChA: track 21.7 -> 10.4 mm
- net /M4_ChA: track 50.9 -> 58.8 mm
- net /L_PWM_3: track 38.1 -> 30.5 mm
- net /M4_ChB: track 50.2 -> 42.7 mm
- net /M3_ChA: track 12.3 -> 19.4 mm
- net /R_PWM_2: track 37.3 -> 34.7 mm
- net /R_PWM_3: track 38.2 -> 35.5 mm
- net /L_PWM_2: track 32.5 -> 30.0 mm
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Other:
- board text added: "12V"
- board text added: "5V GND"
- board text added: "ChB ChA GND 5V M+ M-"
- board text added: "GND"
- board text added: "GND 12V"
- board text added: "GND V12 M- M+"
- board text added: "IN+"
- board text added: "IN-"
- board text added: "Internal Connect"
- board text added: "M+"
- board text added: "M+ M- 12V GND"
- board text added: "M-"
- board text added: "M- M+ 5V GND ChA ChB"
- board text added: "OUT+"
- board text added: "OUT-"

Commit message: order change
Parts:
- moved Ext_GND1 65.2 mm to (84.3, 94.3)
- moved Ext_12V1 3.55 mm to (84.3, 90.0)
- moved Bin1 3.48 mm to (83.6, 81.8)
- moved B-SW_1 3.48 mm to (97.8, 83.4)
- moved BUCK1 3.48 mm to (107.2, 79.1)
- moved Alt_enc2 0.78 mm to (122.3, 34.8)
Connections:
- MD_st1 pad 1: /M+1 -> GND
- MD_st1 pad 2: /M-1 -> /Vin
- MD_st1 pad 3: /Vin -> /M+1
- MD_st1 pad 4: GND -> /M-1
- MD_st2 pad 1: /M+2 -> GND
- MD_st2 pad 2: /M-2 -> /Vin
- MD_st2 pad 3: /Vin -> /M+2
- MD_st2 pad 4: GND -> /M-2
- MD_st3 pad 1: /M+3 -> GND
- MD_st3 pad 2: /M-3 -> /Vin
- MD_st3 pad 3: /Vin -> /M+3
- MD_st3 pad 4: GND -> /M-3
- MD_st4 pad 1: /M+4 -> GND
- MD_st4 pad 2: /M-4 -> /Vin
- MD_st4 pad 3: /Vin -> /M+4
- MD_st4 pad 4: GND -> /M-4
Routing:
- net /Vin: track 191.3 -> 200.7 mm
- net /M+3: track 33.6 -> 42.7 mm
- net /M-2: track 35.5 -> 26.8 mm
- net /M-3: track 32.7 -> 40.4 mm
- net /M-1: track 50.9 -> 45.8 mm
- net /M+1: track 52.0 -> 47.1 mm
- net /M-4: track 11.5 -> 9.44 mm
- net /M+4: track 15.8 -> 14.2 mm
- net Net-(Bin1-Pin_2): track 17.5 -> 16.8 mm
- net /R_PWM_4: track 109.2 -> 108.6 mm
- net GND: vias 93 -> 47
Other:
- board size 116.6 x 82.9 mm -> 116.5 x 82.9 mm
- board text added: "B+"
- board text added: "B-"
- board text added: "B- B+ M+ M-"
- board text added: "M- M+ B+ B-"
- board text removed: "12V"
- board text removed: "GND"
- board text removed: "GND V12 M- M+"
- board text removed: "M+ M- 12V GND"
