File: omni_pcb.kicad_sch (KiCad schematic)
At the start: 25 parts, among them J1 Conn_01x06_Socket, J2 Conn_01x06_Socket, J3 Conn_01x06_Socket, J4 Conn_01x06_Socket, U1 ESP32-DEVKIT-V1

Commit message: pcb layout
Parts:
- removed IMU1: Conn_01x08_Socket, Connector_PinSocket_1.00mm:PinSocket_1x08_P1.00mm_Vertical, symbol Connector:Conn_01x08_Socket
- removed MD_L1, MD_L2, MD_L3, MD_L4, MD_R1, MD_R2, MD_R3, MD_R4: Conn_01x04_Socket, Connector_PinSocket_1.00mm:PinSocket_1x04_P1.00mm_Vertical, symbol Connector:Conn_01x04_Socket
- removed pow-M1, pow-M2, pow-M3, pow-M4, pow-M5, pow-M6, pow-M7, pow-M8: Screw_Terminal_01x02, TerminalBlock:TerminalBlock_Xinya_XY308-2.54-2P_1x02_P2.54mm_Horizontal, symbol Connector:Screw_Terminal_01x02
- added Alt_enc1, Alt_enc2, Alt_enc3, Alt_enc4: Conn_01x06_Socket, Connector_JST:JST_XH_B6B-XH-AM_1x06_P2.50mm_Vertical, symbol Connector:Conn_01x06_Socket
- added ESP_5V1, Ext_12V1, Ext_5V1: TestPoint, Connector_PinHeader_2.54mm:PinHeader_1x01_P2.54mm_Vertical, symbol Connector:TestPoint
- added Ext_GND1: Conn_01x01_Socket, Connector_PinHeader_2.54mm:PinHeader_1x01_P2.54mm_Vertical, symbol Connector:Conn_01x01_Socket
- added H1, H2, H3, H4: MountingHole, MountingHole:MountingHole_2.5mm, symbol Mechanical:MountingHole
- added IMU1: Conn_01x10_Socket, Connector_PinSocket_2.54mm:PinSocket_1x10_P2.54mm_Vertical, symbol Connector:Conn_01x10_Socket
- added MD1, MD2, MD3, MD4: Conn_02x04_Odd_Even, Connector_PinSocket_2.54mm:PinSocket_2x04_P2.54mm_Vertical, symbol Connector_Generic:Conn_02x04_Odd_Even
- added MD_st1, MD_st2, MD_st3, MD_st4: Conn_01x04, Connector_JST:JST_XH_B4B-XH-A_1x04_P2.50mm_Vertical, symbol Connector_Generic:Conn_01x04
- renumbered U1 to ESP1, J1 to Enc1, J2 to Enc2, J3 to Enc3, J4 to Enc4
Connections:
- net +5V: now also Ext_5V1.1, IMU1.10 (Pin_10), MD1.1 (Pin_1), MD1.2 (Pin_2), MD1.5 (Pin_5), MD1.6 (Pin_6), MD2.1 (Pin_1), MD2.2 (Pin_2), MD2.5 (Pin_5), MD2.6 (Pin_6), MD3.1 (Pin_1), MD3.2 (Pin_2), MD3.5 (Pin_5), MD3.6 (Pin_6), MD4.1 (Pin_1), MD4.2 (Pin_2), MD4.5 (Pin_5), MD4.6 (Pin_6)
- net GND: now also Ext_GND1.1 (Pin_1), IMU1.9 (Pin_9), MD_st1.4 (Pin_4), MD_st2.4 (Pin_4), MD_st3.4 (Pin_4), MD_st4.4 (Pin_4)
- net L_PWM_1: now also MD1.8 (Pin_8)
- net L_PWM_2: now also MD2.8 (Pin_8)
- net L_PWM_3: now also MD3.8 (Pin_8)
- net L_PWM_4: now also MD4.8 (Pin_8)
- net M+1: now also MD_st1.1 (Pin_1)
- net M+2: now also MD_st2.1 (Pin_1)
- net M+3: now also MD_st3.1 (Pin_1)
- net M+4: now also MD_st4.1 (Pin_1)
- net M-1: now also MD_st1.2 (Pin_2)
- net M-2: now also MD_st2.2 (Pin_2)
- net M-3: now also MD_st3.2 (Pin_2)
- net M-4: now also MD_st4.2 (Pin_2)
- net R_PWM_1: now also MD1.7 (Pin_7)
- net R_PWM_2: now also MD2.7 (Pin_7)
- net R_PWM_3: now also MD3.7 (Pin_7)
- net R_PWM_4: now also MD4.7 (Pin_7)
- net SCL_imu: now also IMU1.8 (Pin_8)
- net SDA_imu: now also IMU1.7 (Pin_7)
- net Vin: now also Ext_12V1.1, MD_st1.3 (Pin_3), MD_st2.3 (Pin_3), MD_st3.3 (Pin_3), MD_st4.3 (Pin_3)
- net at ESP1.30 (VIN): now also ESP_5V1.1

Commit message: traces
Parts:
- removed ESP_5V1, Ext_12V1, Ext_5V1: TestPoint, Connector_PinHeader_2.54mm:PinHeader_1x01_P2.54mm_Vertical, symbol Connector:TestPoint
- added ESP_5V1: ESP_5V, Connector_Wire:SolderWirePad_1x01_SMD_2x4mm, symbol Connector:Conn_01x01_Socket
- added Ext_12V1: Ext_12V, Connector_Wire:SolderWirePad_1x01_SMD_3x6mm, symbol Connector:Conn_01x01_Socket
- added Ext_5V1: Ext_5V, Connector_Wire:SolderWirePad_1x01_SMD_2x4mm, symbol Connector:Conn_01x01_Socket
- B-SW_1: value 100SP1T1B4M2QE -> SW
- Bin1: value Battery_Terminal -> Bin
- ESP1: value ESP32-DEVKIT-V1 -> ESP
- Ext_GND1: value Conn_01x01_Socket -> Ext_GND; footprint Connector_PinHeader_2.54mm:PinHeader_1x01_P2.54mm_Vertical -> Connector_Wire:SolderWirePad_1x01_SMD_3x6mm
- IMU1: value Conn_01x10_Socket -> IMU
Connections:
- net +5V: now also Alt_enc1.2 (Pin_2), Alt_enc2.2 (Pin_2), Alt_enc3.2 (Pin_2), Alt_enc4.2 (Pin_2), Ext_5V1.1 (Pin_1)
- net GND: now also Alt_enc1.5 (Pin_5), Alt_enc2.5 (Pin_5), Alt_enc3.5 (Pin_5), Alt_enc4.5 (Pin_5)
- net L_PWM_1: now also ESP1.24 (D26); no longer ESP1.22 (D33)
- net L_PWM_2: now also ESP1.22 (D33); no longer ESP1.26 (D14)
- net L_PWM_3: now also ESP1.8 (D5); no longer ESP1.10 (D19)
- net M+1: now also Alt_enc1.1 (Pin_1)
- net M+2: now also Alt_enc2.1 (Pin_1)
- net M+3: now also Alt_enc3.1 (Pin_1)
- net M+4: now also Alt_enc4.1 (Pin_1)
- net M-1: now also Alt_enc1.6 (Pin_6)
- net M-2: now also Alt_enc2.6 (Pin_6)
- net M-3: now also Alt_enc3.6 (Pin_6)
- net M-4: now also Alt_enc4.6 (Pin_6)
- net M1_ChA: now also Alt_enc1.4 (Pin_4)
- net M1_ChB: now also Alt_enc1.3 (Pin_3)
- net M2_ChA: now also Alt_enc2.4 (Pin_4), ESP1.25 (D27); no longer ESP1.24 (D26)
- net M2_ChB: now also Alt_enc2.3 (Pin_3), ESP1.26 (D14); no longer ESP1.23 (D25)
- net M3_ChA: now also Alt_enc3.4 (Pin_4), ESP1.9 (D18); no longer ESP1.8 (D5)
- net M3_ChB: now also Alt_enc3.3 (Pin_3), ESP1.10 (D19); no longer ESP1.5 (D4)
- net M4_ChA: now also Alt_enc4.4 (Pin_4), ESP1.28 (D13); no longer ESP1.27 (D12)
- net M4_ChB: now also Alt_enc4.3 (Pin_3), ESP1.27 (D12); no longer ESP1.28 (D13)
- net R_PWM_1: now also ESP1.23 (D25); no longer ESP1.21 (D32)
- net R_PWM_2: now also ESP1.21 (D32); no longer ESP1.25 (D27)
- net R_PWM_3: now also ESP1.5 (D4); no longer ESP1.9 (D18)
- net Vin: now also Ext_12V1.1 (Pin_1)
- net at ESP1.30 (VIN): now also ESP_5V1.1 (Pin_1)

Commit message: pcb final
Parts:
- Alt_enc1, Alt_enc2, Alt_enc3, Alt_enc4, Enc1, Enc2, Enc3, Enc4: footprint Connector_JST:JST_XH_B6B-XH-AM_1x06_P2.50mm_Vertical -> Connector_JST:JST_XH_B6B-XH-A_1x06_P2.50mm_Vertical
Connections:
- net +5V: no longer Alt_enc1.2 (Pin_2), Alt_enc2.2 (Pin_2), Alt_enc3.2 (Pin_2), Alt_enc4.2 (Pin_2), MD1.2 (Pin_2), MD2.2 (Pin_2), MD3.2 (Pin_2), MD4.2 (Pin_2)
- net GND: now also MD1.2 (Pin_2), MD2.2 (Pin_2), MD3.2 (Pin_2), MD4.2 (Pin_2); no longer Alt_enc1.5 (Pin_5), Alt_enc2.5 (Pin_5), Alt_enc3.5 (Pin_5), Alt_enc4.5 (Pin_5)
- net L_PWM_2: now also ESP1.20 (D35); no longer ESP1.22 (D33)
- net M+1: no longer Alt_enc1.1 (Pin_1)
- net M+2: no longer Alt_enc2.1 (Pin_1)
- net M+3: no longer Alt_enc3.1 (Pin_1)
- net M+4: no longer Alt_enc4.1 (Pin_1)
- net M-1: no longer Alt_enc1.6 (Pin_6)
- net M-2: no longer Alt_enc2.6 (Pin_6)
- net M-3: no longer Alt_enc3.6 (Pin_6)
- net M-4: no longer Alt_enc4.6 (Pin_6)
- net M1_ChA: now also ESP1.21 (D32); no longer Alt_enc1.4 (Pin_4), ESP1.20 (D35)
- net M1_ChB: now also ESP1.22 (D33); no longer Alt_enc1.3 (Pin_3), ESP1.19 (D34)
- net M2_ChA: no longer Alt_enc2.4 (Pin_4)
- net M2_ChB: no longer Alt_enc2.3 (Pin_3)
- net M3_ChA: no longer Alt_enc3.4 (Pin_4)
- net M3_ChB: no longer Alt_enc3.3 (Pin_3)
- net M4_ChA: no longer Alt_enc4.4 (Pin_4)
- net M4_ChB: no longer Alt_enc4.3 (Pin_3)
- net R_PWM_2: now also ESP1.19 (D34); no longer ESP1.21 (D32)
Other:
- moved on the sheet: Alt_enc1, Alt_enc2, Alt_enc3, Alt_enc4

Commit message: pin changes
Connections:
- net L_PWM_2: now also ESP1.22 (D33); no longer ESP1.20 (D35)
- net L_PWM_3: now also ESP1.5 (D4); no longer ESP1.8 (D5)
- net L_PWM_4: now also ESP1.3 (D15); no longer ESP1.4 (D2)
- net M1_ChA: now also ESP1.19 (D34); no longer ESP1.21 (D32)
- net M1_ChB: now also ESP1.20 (D35); no longer ESP1.22 (D33)
- net M3_ChA: now also ESP1.10 (D19); no longer ESP1.9 (D18)
- net M3_ChB: now also ESP1.15 (D23); no longer ESP1.10 (D19)
- net M4_ChA: now also ESP1.27 (D12); no longer ESP1.28 (D13)
- net M4_ChB: now also ESP1.9 (D18); no longer ESP1.27 (D12)
- net R_PWM_2: now also ESP1.21 (D32); no longer ESP1.19 (D34)
- net R_PWM_3: now also ESP1.4 (D2); no longer ESP1.5 (D4)
- net R_PWM_4: now also ESP1.28 (D13); no longer ESP1.3 (D15)
Changed lines of the file:
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@@
-	(wire
-		(pts
-			(xy 123.19 76.2) (xy 129.54 76.2)
-		)
-		(stroke
-			(width 0)
-			(type default)
-		)
-	)
 	(wire
 		(pts
@@
 		(pts
 			(xy 217.17 40.64) (xy 222.25 40.64)
+		)
+		(stroke
+			(width 0)
+			(type default)
+		)
+	)
+	(wire
+		(pts
+			(xy 160.02 73.66) (xy 166.37 73.66)
 		)
 		(stroke
@@
 	)
 	(label "R_PWM_3"
-		(at 123.19 73.66 180)
+		(at 123.19 71.12 180)
 		(effects
 			(font
@@
 	)
 	(label "L_PWM_2"
-		(at 166.37 88.9 0)
+		(at 166.37 86.36 0)
 		(effects
 			(font
@@
 	)
 	(label "M3_ChA"
-		(at 123.19 88.9 180)
+		(at 123.19 91.44 180)
 		(effects
 			(font
@@
 	)
 	(label "M4_ChA"
-		(at 123.19 81.28 180)
+		(at 123.19 78.74 180)
 		(effects
 			(font
@@
 	)
 	(label "M1_ChA"
-		(at 166.37 83.82 0)
+		(at 166.37 91.44 0)
 		(effects
 			(font
@@
 	)
 	(label "R_PWM_2"
-		(at 166.37 91.44 0)
+		(at 166.37 83.82 0)
 		(effects
 			(font
@@
 	)
 	(label "M4_ChB"
-		(at 123.19 78.74 180)
+		(at 123.19 88.9 180)
 		(effects
 			(font
@@
 	)
 	(label "R_PWM_4"
-		(at 123.19 86.36 180)
+		(at 123.19 81.28 180)
 		(effects
 			(font
@@
 	)
 	(label "M3_ChB"
-		(at 123.19 91.44 180)
-		(effects
-			(font
-				(size 1.27 1.27)
-			)
-			(justify right bottom)
+		(at 166.37 73.66 0)
+		(effects
+			(font
+				(size 1.27 1.27)
+			)
+			(justify left bottom)
 		)
 	)
@@
 	)
 	(label "L_PWM_4"
-		(at 123.19 71.12 180)
+		(at 123.19 86.36 180)
 		(effects
 			(font
@@
 	)
 	(label "M1_ChB"
-		(at 166.37 86.36 0)
+		(at 166.37 88.9 0)
 		(effects
 			(font
@@
 	)
 	(label "L_PWM_3"
-		(at 123.19 76.2 180)
-		(effects
-			(font
+		(at 123.19 73.66 180)
+		(effects
+			(font

Commit message: order change
Connections:
- net GND: now also MD_st1.1 (Pin_1), MD_st2.1 (Pin_1), MD_st3.1 (Pin_1), MD_st4.1 (Pin_1); no longer MD_st1.4 (Pin_4), MD_st2.4 (Pin_4), MD_st3.4 (Pin_4), MD_st4.4 (Pin_4)
- net M+1: now also MD_st1.3 (Pin_3); no longer MD_st1.1 (Pin_1)
- net M+2: now also MD_st2.3 (Pin_3); no longer MD_st2.1 (Pin_1)
- net M+3: now also MD_st3.3 (Pin_3); no longer MD_st3.1 (Pin_1)
- net M+4: now also MD_st4.3 (Pin_3); no longer MD_st4.1 (Pin_1)
- net M-1: now also MD_st1.4 (Pin_4); no longer MD_st1.2 (Pin_2)
- net M-2: now also MD_st2.4 (Pin_4); no longer MD_st2.2 (Pin_2)
- net M-3: now also MD_st3.4 (Pin_4); no longer MD_st3.2 (Pin_2)
- net M-4: now also MD_st4.4 (Pin_4); no longer MD_st4.2 (Pin_2)
- net Vin: now also MD_st1.2 (Pin_2), MD_st2.2 (Pin_2), MD_st3.2 (Pin_2), MD_st4.2 (Pin_2); no longer MD_st1.3 (Pin_3), MD_st2.3 (Pin_3), MD_st3.3 (Pin_3), MD_st4.3 (Pin_3)
Changed lines of the file:
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@@
 	)
 	(label "M-2"
-		(at 64.77 160.02 180)
+		(at 64.77 165.1 180)
 		(effects
 			(font
@@
 	)
 	(label "M-3"
-		(at 101.6 140.97 180)
+		(at 101.6 146.05 180)
 		(effects
 			(font
@@
 	)
 	(label "M+3"
-		(at 101.6 138.43 180)
+		(at 101.6 143.51 180)
 		(effects
 			(font
@@
 	)
 	(label "Vin"
-		(at 64.77 143.51 180)
+		(at 64.77 140.97 180)
 		(effects
 			(font
@@
 	)
 	(label "M+4"
-		(at 101.6 157.48 180)
+		(at 101.6 162.56 180)
 		(effects
 			(font
@@
 	)
 	(label "M-1"
-		(at 64.77 140.97 180)
+		(at 64.77 146.05 180)
 		(effects
 			(font
@@
 	)
 	(label "Vin"
-		(at 101.6 143.51 180)
+		(at 101.6 140.97 180)
 		(effects
 			(font
@@
 	)
 	(label "Vin"
-		(at 101.6 162.56 180)
+		(at 101.6 160.02 180)
 		(effects
 			(font
@@
 	)
 	(label "M-4"
-		(at 101.6 160.02 180)
+		(at 101.6 165.1 180)
 		(effects
 			(font
@@
 	)
 	(label "Vin"
-		(at 64.77 162.56 180)
+		(at 64.77 160.02 180)
 		(effects
 			(font
@@
 	)
 	(label "M+2"
-		(at 64.77 157.48 180)
+		(at 64.77 162.56 180)
 		(effects
 			(font
@@
 	)
 	(label "M+1"
-		(at 64.77 138.43 180)
+		(at 64.77 143.51 180)
 		(effects
 			(font
@@
 	(symbol
 		(lib_id "power:GND")
-		(at 101.6 165.1 270)
+		(at 101.6 157.48 270)
 		(mirror x)
 		(unit 1)
@@
 		(dnp no)
 		(property "Reference" "#PWR028"
-			(at 95.25 165.1 0)
+			(at 95.25 157.48 0)
 			(effects
 				(font
@@
 		)
 		(property "Value" "GND"
-			(at 98.298 165.1 90)
+			(at 98.298 157.48 90)
 			(effects
 				(font
@@
 		)
 		(property "Footprint" ""
-			(at 101.6 165.1 0)
+			(at 101.6 157.48 0)
 			(effects
 				(font
@@
 		)
 		(property "Datasheet" ""
-			(at 101.6 165.1 0)
+			(at 101.6 157.48 0)
 			(effects
 				(font
@@
 		)
 		(property "Description" "Power symbol creates a global label with name \"GND\" , ground"
-			(at 101.6 165.1 0)
+			(at 101.6 157.48 0)
 			(effects
 				(font
@@
 	(symbol
 		(lib_id "power:GND")
-		(at 64.77 165.1 270)
+		(at 64.77 157.48 270)
 		(mirror x)
 		(unit 1)
@@
 		(dnp no)
 		(property "Reference" "#PWR019"
-			(at 58.42 165.1 0)
+			(at 58.42 157.48 0)
 			(effects
 				(font
@@
 		)
 		(property "Value" "GND"
-			(at 61.468 165.1 90)
+			(at 61.468 157.48 90)
 			(effects
 				(font
@@
 		)
 		(property "Footprint" ""
-			(at 64.77 165.1 0)
+			(at 64.77 157.48 0)
 			(effects
 				(font
@@
 		)
 		(property "Datasheet" ""
-			(at 64.77 165.1 0)
+			(at 64.77 157.48 0)
 			(effects
 				(font
@@
 		)
 		(property "Description" "Power symbol creates a global label with name \"GND\" , ground"
-			(at 64.77 165.1 0)
+			(at 64.77 157.48 0)
 			(effects
 				(font
@@
 	(symbol
 		(lib_id "power:GND")
-		(at 64.77 146.05 270)
+		(at 64.77 138.43 270)
 		(mirror x)
 		(unit 1)
@@
 		(dnp no)
 		(property "Reference" "#PWR01"
-			(at 58.42 146.05 0)
+			(at 58.42 138.43 0)
 			(effects
 				(font
@@
 		)
 		(property "Value" "GND"
-			(at 61.468 146.05 90)
+			(at 61.468 138.43 90)
 			(effects
 				(font
@@
 		)
 		(property "Footprint" ""
-			(at 64.77 146.05 0)
+			(at 64.77 138.43 0)
 			(effects
 				(font
@@
 		)
 		(property "Datasheet" ""
-			(at 64.77 146.05 0)
+			(at 64.77 138.43 0)
 			(effects
 				(font
@@
 		)
 		(property "Description" "Power symbol creates a global label with name \"GND\" , ground"
-			(at 64.77 146.05 0)
+			(at 64.77 138.43 0)
 			(effects
 				(font
@@
 	(symbol
 		(lib_id "power:GND")
-		(at 101.6 146.05 270)
+		(at 101.6 138.43 270)
 		(mirror x)
 		(unit 1)
@@
 		(dnp no)
 		(property "Reference" "#PWR020"
-			(at 95.25 146.05 0)
+			(at 95.25 138.43 0)
 			(effects
 				(font
@@
 		)
 		(property "Value" "GND"
-			(at 98.298 146.05 90)
+			(at 98.298 138.43 90)
 			(effects
 				(font
@@
 		)
 		(property "Footprint" ""
-			(at 101.6 146.05 0)
+			(at 101.6 138.43 0)
 			(effects
 				(font
@@
 		)
 		(property "Datasheet" ""
-			(at 101.6 146.05 0)
+			(at 101.6 138.43 0)
 			(effects
 				(font
@@
 		)
 		(property "Description" "Power symbol creates a global label with name \"GND\" , ground"
-			(at 101.6 146.05 0)
+			(at 101.6 138.43 0)
 			(effects
 				(font
